File: MeasurementCard.sch (KiCad schematic (older format))
At the start: 218 parts, among them J1 Conn_01x05, J10 Conn_01x01, J13 Conn_01x01, J14 Conn_01x01, J17 Conn_01x03, J18 Conn_01x02, J2 Conn_01x02, J3 Conn_01x13, J4 Conn_01x03, J5 Conn_01x03, J6 Conn_01x03, J7 Conn_01x03, J8 Conn_01x13, J9 Conn_01x01, Q1 BSS138, Q10 BSS138, Q11 BSS138, Q12 BSS138, Q13 NSV1C201MZ4, Q14 BSS138, Q15 BSS138, Q16 BSS138, Q17 BSS138, Q18 BSS138, Q19 BSS138, Q2 BSS138, Q20 BSS138, Q21 BSS138, Q22 BSS138, Q23 BSS138, Q24 BSS138, Q25 BSS138, Q26 NSV1C201MZ4, Q3 BSS138, Q4 BSS138, Q5 BSS138, Q6 BSS138, Q7 BSS138, Q8 BSS138, Q9 BSS138, T1 HX1188NL, T2 HX1188NL, U1 LTC6804-1, U2 LTC6804-1

Commit message: added db25 + thermistor support
Parts:
- removed J3, J8: Conn_01x13, Connector_JST:JST_XH_S13B-XH-A_1x13_P2.50mm_Horizontal, symbol MeasurementCard-rescue:Conn_01x13-conn-onestacker_butbetter-rescue-twostacker-r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
- added J11, J8: Conn_01x02, Connector_JST:JST_XH_S2B-XH-A_1x02_P2.50mm_Horizontal, symbol Connector_Generic:Conn_01x02
- added J3: Conn_01x25, Connector_Dsub:DSUB-25_Male_Horizontal_P2.77x2.84mm_EdgePinOffset7.70mm_Housed_MountingHolesOffset9.12mm, symbol Connector_Generic:Conn_01x25
- added R111, R112: 10k, Resistor_SMD:R_0805_2012Metric_Pad1.15x1.40mm_HandSolder, symbol Device:R_Small
- T1, T2: symbol HX1188NL:HX1188NL -> MeasurementCard-rescue:HX1188NL-HX1188NL
- U1, U2: symbol 6804-1:LTC6804-1 -> MeasurementCard-rescue:LTC6804-1-6804-1
Connections:
- net GND: now also J3.25 (Pin_25), J8.2 (Pin_2)
- net GNDA: now also Q12.2 (S), R48.2, R49.2, R50.2, J11.2 (Pin_2), J3.13 (Pin_13)
- net VTEMP1: now reaches U1.27 (GPIO1)
- net VTEMP1: now also J8.1 (Pin_1), R111.2
- net VREF2_1: now reaches C1.1, U1.34 (VREF2)
- net VREF2_1: now also C35.1, U2.35 (VREF1), R111.1
- net at Q1.2 (S), R4.2, R5.2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: now also J3.24 (Pin_24)
- net at Q2.2 (S), R11.1, R8.2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: now also J3.23 (Pin_23)
- net at Q3.2 (S), R12.2, R13.2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: now also J3.22 (Pin_22)
- net at Q4.2 (S), R16.2, R17.2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: now also J3.21 (Pin_21)
- net at Q5.2 (S), R20.2, R21.2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: now also J3.20 (Pin_20)
- net at Q6.2 (S), R24.2, R25.2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: now also J3.19 (Pin_19)
- net at Q7.2 (S), R28.2, R29.2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: now also J3.18 (Pin_18)
- net at Q8.2 (S), R32.2, R33.2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: now also J3.17 (Pin_17)
- net at Q9.2 (S), R36.2, R37.2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: now also J3.16 (Pin_16)
- net at Q10.2 (S), R40.2, R41.2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: now also J3.15 (Pin_15)
- net at Q11.2 (S), R44.2, R45.2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: now also J3.14 (Pin_14)
- net VTEMP2: now reaches U2.27 (GPIO1)
- net VTEMP2: now also J11.1 (Pin_1), R112.2
- net at Q25.2 (S), R106.2, R67.2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: now also J3.12 (Pin_12)
- net at Q24.2 (S), R105.2, R66.2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: now also J3.11 (Pin_11)
- net at Q23.2 (S), R104.2, R65.2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: now also J3.10 (Pin_10)
- net at Q22.2 (S), R103.2, R64.2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: now also J3.9 (Pin_9)
- net at Q21.2 (S), R102.2, R63.2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: now also J3.8 (Pin_8)
- net at Q20.2 (S), R101.2, R62.2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: now also J3.7 (Pin_7)
- net at Q19.2 (S), R100.2, R61.2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: now also J3.6 (Pin_6)
- net at Q18.2 (S), R60.2, R72.1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: now also J3.5 (Pin_5)
- net at Q17.2 (S), R59.2, R71.1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: now also J3.4 (Pin_4)
- net at Q16.2 (S), R58.2, R70.1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: now also J3.3 (Pin_3)
- net at Q15.2 (S), R57.2, R69.1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: now also J3.2 (Pin_2)
- net at Q14.2 (S), R93.2, R94.2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: now also J3.1 (Pin_1)
- new net VREF2_2: R112.1
Other:
- moved on the sheet: C21, C22, C23, C24, C25, C26, C27, C28, C29, C30, C31, C32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
